File: PCB/Pet_sitting.kicad_pcb (KiCad board)
At the start: 2 copper layers, 91.4 x 46.5 mm, 15 parts, among them IC1 ESP32-CAM, J1 Conn_01x02, J2 Conn_01x02_Female, J3 Conn_01x02, J4 Conn_01x02, J5 Conn_01x06_Female, M1 Motor_Servo, U1 DFR0299, U2 L293D, U3 LM1117-5.0

Commit message: Add files via upload
Parts:
- added J6: Conn_01x02_Female, Connector_PinSocket_2.54mm:PinSocket_1x02_P2.54mm_Vertical, F.Cu at (163.3, 91.2)
- added J7: Conn_01x02_Female, Connector_PinSocket_2.54mm:PinSocket_1x02_P2.54mm_Vertical, F.Cu at (168.4, 91.2)
- added REF**: MountingHole_2.1mm, MountingHole:MountingHole_2.1mm, F.Cu at (199.9, 117.3)
- added REF**: MountingHole_2.1mm, MountingHole:MountingHole_2.1mm, F.Cu at (115.3, 117.1)
- added REF**: MountingHole_2.1mm, MountingHole:MountingHole_2.1mm, F.Cu at (115.1, 73.2)
- added REF**: MountingHole_2.1mm, MountingHole:MountingHole_2.1mm, F.Cu at (199.9, 73.2)
- moved R1 5.78 mm to (172.5, 94.2)
- moved R2 5.78 mm to (172.5, 90.7)
- moved Speaker 4.17 mm to (172.0, 99.6)
- moved J2 4.12 mm to (163.6, 82.8), turned to 90 degrees
- moved J5 3.22 mm to (163.3, 78.0)
- moved U1 3.06 mm to (182.1, 78.0)
- renumbered LS1 to Speaker
Connections:
- R1 pad 1: Net-(IC1-Pad15) -> Net-(R1-Pad1)
- R2 pad 1: Net-(IC1-Pad14) -> Net-(R2-Pad1)
Routing:
- net GND: track 173.7 -> 11.6 mm, vias 3 -> 1
- net Net-(C2-Pad1): track 286.7 -> 209.0 mm, vias 1 -> 0
- net Net-(IC1-Pad3): track 67.5 -> 42.9 mm, vias 0 -> 1
- net Net-(IC1-Pad4): track 78.2 -> 62.4 mm, vias 0 -> 1
- net Net-(C1-Pad1): track 105.9 -> 115.7 mm
- net Net-(LS1-Pad1): track 12.0 -> 20.8 mm
- net Net-(R1-Pad2): track 12.4 -> 20.9 mm
- net Net-(IC1-Pad16): track 27.0 -> 34.2 mm
- net Net-(IC1-Pad12): track 7.65 -> 13.5 mm
- net Net-(R2-Pad2): track 6.77 -> 11.9 mm
- net Net-(R2-Pad1): track 0.00 -> 4.28 mm
- net Net-(R1-Pad1): track 0.00 -> 4.27 mm
- net Net-(IC1-Pad15): track 27.2 -> 30.2 mm
- net Net-(IC1-Pad6): track 77.0 -> 74.4 mm
- net Net-(IC1-Pad11): track 7.65 -> 9.87 mm
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- added copper zone on F.Cu, net GND
Other:
- board size 91.4 x 46.5 mm -> 91.4 x 50.8 mm
- board text added: "+"
- board text added: "-"
- board text added: "GND"
- board text added: "Motor"
- board text added: "RX"
- board text added: "TX"
- board text added: "VCC"

Commit message: Add files via upload
Parts:
- removed J7: Conn_01x02_Female, Connector_PinSocket_2.54mm:PinSocket_1x02_P2.54mm_Vertical
- removed the REF** at (199.9, 117.3)
- removed the REF** at (115.3, 117.1)
- added REF**: MountingHole_2.1mm, MountingHole:MountingHole_2.1mm, F.Cu at (115.1, 117.3)
- added REF**: MountingHole_2.1mm, MountingHole:MountingHole_2.1mm, F.Cu at (199.9, 117.6)
- J6: value Conn_01x02_Female -> Conn_02x02_Odd_Even; footprint Connector_PinSocket_2.54mm:PinSocket_1x02_P2.54mm_Vertical -> Connector_PinHeader_2.54mm:PinHeader_2x02_P2.54mm_Vertical
- moved R1 4.11 mm to (170.9, 90.4)
- moved Speaker 3.60 mm to (168.4, 99.6), turned to 0 degrees
- moved R2 2.98 mm to (170.9, 93.2)
- moved J6 1.12 mm to (164.3, 90.7)
Connections:
- IC1 pad 12: Net-(IC1-Pad12) -> GND
- IC1 pad 16: Net-(IC1-Pad16) -> GND
- J2 pad 2: Net-(IC1-Pad12) -> GND
- J5 pad 1: Net-(IC1-Pad16) -> GND
- J6 pad 1: Net-(IC1-Pad14) -> Net-(IC1-Pad15)
- J6 pad 2: Net-(IC1-Pad15) -> Net-(R1-Pad1)
Routing:
- net Net-(IC1-Pad16): track 34.2 -> 0.00 mm
- net Net-(IC1-Pad12): track 13.5 -> 0.00 mm
- net Net-(U1-Pad2): track 20.9 -> 12.4 mm
- net Net-(IC1-Pad14): track 25.7 -> 32.8 mm, vias 0 -> 2
- net Net-(LS1-Pad2): track 16.6 -> 11.7 mm
- net Net-(IC1-Pad15): track 30.2 -> 28.1 mm
- net Net-(LS1-Pad1): track 20.8 -> 19.0 mm
- net Net-(U1-Pad3): track 11.9 -> 12.7 mm
